Commit message: Added lidar, imu, and camera

File: catkin_ws/src/twirtee_description/urdf/macros.xacro (robot description, xacro)
@@ -33,11 +33,20 @@
       <cylinder length="${wheelWidth}" radius="${wheelRadius}"/>
     </geometry>
-    <material name="black"/>
+    <material name="cyan"/>
+  </visual>
+  <visual>
+    <origin xyz="0 ${motorAxisWidth/2.0-wheelWidth/2.0} 0 " rpy="0 ${PI/2} ${PI/2}" />
+    <geometry>
+      <cylinder length="${motorAxisWidth}" radius="${motorAxisRadius}"/>
+    </geometry>
+    <material name="red">
+		<color rgba="1.0 0.0 0.0 1.0"/>
+	</material>
   </visual>
 </link>
-<joint name="${lr}_wheel_hinge" type="continuous">
-  <parent link="level0"/>
+<joint name="${lr}_motor_${lr}wheel_joint" type="continuous">
+  <parent link="${lr}_motor"/>
   <child link="${lr}_wheel"/>
-  <origin xyz="${floor0Length/2-wheelXOffset} ${tY*wheelWidth/2+tY*floor0Width/2} ${-wheelFloor0Offset-floor0Heigth/2}" rpy="0 0 0" />
+  <origin xyz="0 ${-motorC1Width/2.0-motorC3Width-motorFixtVHeigth} ${-wheelOffset}" rpy="0 0 0" />
   <axis xyz="0 1 0" rpy="0 0 0" />
   <limit effort="100" velocity="100"/>
@@ -46,5 +55,24 @@
 </xacro:macro>
 <!-- - - - - - - - - - - -->
-<!--      Motors         -->
+<!--   CASTER WHEELS     -->
+<!-- - - - - - - - - - - -->
+<xacro:macro name="caster" params="lr tY">
+<link name="${lr}_caster">
+   <visual>
+    <origin xyz="0 0 0" rpy="0 0 0"/>
+    <geometry>
+      <sphere radius="${casterRadius}"/>
+    </geometry>
+    <material name="red"/>
+  </visual>
+</link>
+<joint name="floor0_${lr}_caster_joint" type="fixed">
+	<origin xyz="${-floor0Length/2.0+0.04} ${tY*0.05} ${-floor0Heigth/2-motorFixtVLength/2.0-motorFixtVOffset-wheelOffset-wheelRadius+casterRadius}" rpy="0 0 0" />
+  <parent link="floor0"/>
+  <child link="${lr}_caster"/>
+</joint>
+</xacro:macro>
+<!-- - - - - - - - - - - -->
+<!--      MOTORS         -->
 <!-- - - - - - - - - - - -->
 <xacro:macro name="motor" params="lr tY">
@@ -53,9 +81,78 @@
     <origin xyz="0 0 0" rpy="0 ${PI/2} ${PI/2}" />
     <geometry>
-      <cylinder length="${wheelWidth}" radius="${wheelRadius}"/>
+      <cylinder length="${motorC1Width}" radius="${motorC1Radius}"/>
     </geometry>
     <material name="black"/>
   </visual>
+  <visual>
+    <origin xyz="0 ${motorC1Width/2+motorC2Width/2.0} 0" rpy="0 ${PI/2} ${PI/2}" />
+    <geometry>
+      <cylinder length="${motorC2Width}" radius="${motorC2Radius}"/>
+    </geometry>
+    <material name="green">
+		<color rgba="0.0 1.0 0.0 1.0"/>
+	</material>
+  </visual>
+  <visual>
+    <origin xyz="0 ${-motorC1Width/2.0-motorC3Width/2.0} ${-wheelOffset}" rpy="0 ${PI/2} ${PI/2}" />
+    <geometry>
+      <cylinder length="${motorC3Width}" radius="${motorC3Radius}"/>
+    </geometry>
+    <material name="blue">
+		<color rgba="0.0 0.0 1.0 1.0"/>
+	</material>
+  </visual>
+  <visual>
+    <origin xyz="0 ${-motorC1Width/2.0-motorFixtVHeigth/2.0} ${motorFixtVOffset}" rpy="0 ${PI/2} ${PI/2}" />
+    <geometry>
+		<box size="${motorFixtVLength} ${motorFixtVWidth} ${motorFixtVHeigth}" />
+    </geometry>
+    <material name="red">
+		<color rgba="1.0 0.0 0.0 1.0"/>
+	</material>
+  </visual>
+  <visual>
+    <origin xyz="0 ${-motorC1Width/2.0+motorFixtHLength/2.0} ${motorFixtVLength/2.0-motorFixtHHeigth/2.0+motorFixtVOffset}" rpy="0 ${PI/2} ${PI/2}" />
+    <geometry>
+		<box size="${motorFixtHHeigth} ${motorFixtHWidth} ${motorFixtHLength}" />
+    </geometry>
+    <material name="red">
+		<color rgba="1.0 0.0 0.0 1.0"/>
+	</material>
+  </visual>
 </link>
+<joint name="l0_${lr}_motor_joint" type="fixed">
+  <parent link="floor0"/>
+  <child link="${lr}_motor"/>
+  <origin xyz="${floor0Length/2-wheelXOffset} ${tY*floor0Width/2} ${-floor0Heigth/2-motorFixtVLength/2.0-motorFixtVOffset}" rpy="0 0 ${(tY+1)*PI/2.0}" />
+  <axis xyz="0 1 0" rpy="0 0 0" />
+  <limit effort="100" velocity="100"/>
+  <joint_properties damping="0.0" friction="0.0"/>
+</joint>
+</xacro:macro>
+<!-- - - - - - - - - - - -->
+<!--      Pilars         -->
+<!-- - - - - - - - - - - -->
+<xacro:macro name="f0Pilar" params="tX tY">
+  <visual>
+    <origin xyz="${tX*0.14} ${tY*0.0925} ${floor0Heigth/2.0+spacer01Width/2.0}" rpy="0 0 0" />
+    <geometry>
+      <cylinder length="${spacer01Width}" radius="${spacerRadius}"/>
+    </geometry>
+    <material name="green">
+		<color rgba="0.0 1.0 0.0 1.0"/>
+	</material>
+  </visual>
+</xacro:macro>
+<xacro:macro name="f1Pilar" params="tX tY">
+  <visual>
+    <origin xyz="${tX*0.14} ${tY*0.0925} ${floor1Heigth/2.0+spacer12Width/2.0}" rpy="0 0 0" />
+    <geometry>
+      <cylinder length="${spacer12Width}" radius="${spacerRadius}"/>
+    </geometry>
+    <material name="green">
+		<color rgba="0.0 1.0 0.0 1.0"/>
+	</material>
+  </visual>
 </xacro:macro>
 </robot>

File: catkin_ws/src/twirtee_description/urdf/twirtee.urdf (robot description, URDF)
Before this commit: robot twirtee, 6 links, 5 joints
Links:
- removed link level0
- removed link level1
- removed link level2
- added link cam; visual box size=0.02 0.02 0.02
- added link floor0; visual box size=0.3 0.2 0.003; visual cylinder length=0.06 radius=0.002
- added link floor1; visual box size=0.35 0.25 0.003; visual cylinder length=0.05 radius=0.002
- added link floor2; visual box size=0.35 0.25 0.003
- added link imu; visual box size=0.01 0.005 0.01
- added link left_caster; visual sphere radius=0.02
- added link left_motor; visual box size=0.003 0.04 0.04; visual box size=0.045 0.04 0.003
- added link lidarbase; visual cylinder length=0.035 radius=0.035
- added link lidarhead; visual cylinder length=0.02 radius=0.035
- added link right_caster; visual sphere radius=0.02
- added link right_motor; visual box size=0.003 0.04 0.04; visual box size=0.045 0.04 0.003
- link left_wheel: geometry visual cylinder length=0.01 radius=0.032; visual cylinder length=0.0145 radius=0.003
- link right_wheel: geometry visual cylinder length=0.01 radius=0.032; visual cylinder length=0.0145 radius=0.003
Joints:
- removed joint l0l1_joint
- removed joint l1l2_joint
- removed joint left_wheel_hinge
- removed joint right_wheel_hinge
- added joint f0f1_joint: type fixed, parent floor0, child floor1, origin xyz= 0.0 0.0 0.0615 rpy=0 0 0
- added joint f1_imu_joint: type fixed, parent floor1, child imu, origin xyz= 0.0 0.0 0.0065 rpy=0 0 0
- added joint f1f2_joint: type fixed, parent floor1, child floor2, origin xyz= 0.0 0.0 0.0515 rpy=0 0 0
- added joint f2_cam_joint: type fixed, parent floor2, child cam, origin xyz= 0.175 0.05 0.0315 rpy=0 0.3 0
- added joint f2_lidarbase_joint: type fixed, parent floor2, child lidarbase, origin xyz= 0.14 0.0 0.019 rpy=0 0 0
- added joint floor0_left_caster_joint: type fixed, parent floor0, child left_caster, origin xyz=-0.11 0.05 -0.045 rpy=0 0 0
- added joint floor0_right_caster_joint: type fixed, parent floor0, child right_caster, origin xyz=-0.11 -0.05 -0.045 rpy=0 0 0
- added joint l0_left_motor_joint: type fixed, parent floor0, child left_motor, origin xyz=0.1 0.1 -0.026 rpy=0 0 3.14159265359, axis 0 1 0, limit effort=100 velocity=100
- added joint l0_right_motor_joint: type fixed, parent floor0, child right_motor, origin xyz=0.1 -0.1 -0.026 rpy=0 0 0.0, axis 0 1 0, limit effort=100 velocity=100
- added joint left_motor_leftwheel_joint: type continuous, parent left_motor, child left_wheel, origin xyz=0 -0.01975 -0.007 rpy=0 0 0, axis 0 1 0, limit effort=100 velocity=100
- added joint lidarbase_head_joint: type continuous, parent lidarbase, child lidarhead, origin xyz= 0.0 0.0 0.0275 rpy=0 0 0, axis 0.0 0.0 1.0
- added joint right_motor_rightwheel_joint: type continuous, parent right_motor, child right_wheel, origin xyz=0 -0.01975 -0.007 rpy=0 0 0, axis 0 1 0, limit effort=100 velocity=100
- joint base_joint: child level0 -> floor0; origin xyz=0 0 0.0665 rpy=0 0 0 -> xyz=0 0 0.068 rpy=0 0 0

File: catkin_ws/src/twirtee_description/urdf/twirtee.xacro (robot description, xacro)
@@ -16,12 +16,12 @@
   <xacro:property name="spacer01Width" 	value="0.060"/>
   <xacro:property name="spacer01Mass" 	value="1"/>
-  <xacro:property name="floor1Length" 	value="0.300"/>
-  <xacro:property name="floor1Width" 	value="0.200"/>
+  <xacro:property name="floor1Length" 	value="0.350"/>
+  <xacro:property name="floor1Width" 	value="0.250"/>
   <xacro:property name="floor1Heigth" 	value="0.003"/>
   <xacro:property name="floor1Mass" 	value="1"/>
   <xacro:property name="spacer12Width" 	value="0.050"/>
   <xacro:property name="spacer12Mass" 	value="1"/>
-  <xacro:property name="floor2Length" 	value="0.30"/>
-  <xacro:property name="floor2Width" 	value="0.20"/>
+  <xacro:property name="floor2Length" 	value="0.350"/>
+  <xacro:property name="floor2Width" 	value="0.250"/>
   <xacro:property name="floor2Heigth" 	value="0.003"/>
   <xacro:property name="floor2Mass" 	value="1"/>
@@ -31,24 +31,48 @@
   <xacro:property name="wheelRadius" 	value="0.032"/>
   <xacro:property name="wheelMass" 		value="5"/>
-  <xacro:property name="wheelExcen" 	value="0.007"/>
+  <xacro:property name="wheelOffset" 	value="0.007"/>
   <xacro:property name="wheelFixtOffset" 	value="0.030"/>
   <xacro:property name="wheelFloor0Offset" 	value="${wheelFixtOffset+motorFixtHHeigth}"/>
   <xacro:property name="wheelXOffset" 	value="0.05"/>
-  <xacro:property name="motorAxisWidth" 	value="0.0045"/>
+  <xacro:property name="motorAxisWidth" 	value="0.0145"/>
   <xacro:property name="motorAxisRadius" 	value="0.003"/>
   <xacro:property name="motorAxisMass" 		value="5"/>
-  <xacro:property name="motorWidth" 	value="0.0445"/>
-  <xacro:property name="motorRadius" 	value="0.0185"/>
-  <xacro:property name="motorMass" 		value="5"/>
-  <xacro:property name="motorFixtVLength" 	value="0.30"/>
-  <xacro:property name="motorFixtVWidth" 	value="0.20"/>
+  <xacro:property name="motorC1Width" 	value="0.0215"/>
+  <xacro:property name="motorC1Radius" 	value="0.0185"/>
+  <xacro:property name="motorC1Mass" 		value="5"/>
+  <xacro:property name="motorC2Width" 	value="0.0230"/>
+  <xacro:property name="motorC2Radius" 	value="0.0164"/>
+  <xacro:property name="motorC2Mass" 		value="5"/>
+  <xacro:property name="motorC3Width" 	value="0.006"/>
+  <xacro:property name="motorC3Radius" 	value="0.006"/>
+  <xacro:property name="motorC3Mass" 		value="5"/>
+  <xacro:property name="motorFixtVLength" 	value="0.045"/>
+  <xacro:property name="motorFixtVWidth" 	value="0.040"/>
   <xacro:property name="motorFixtVHeigth" 	value="0.003"/>
   <xacro:property name="motorFixtVMass" 	value="1"/>
-  <xacro:property name="motorFixtHLength" 	value="0.30"/>
-  <xacro:property name="motorFixtHWidth" 	value="0.20"/>
+  <xacro:property name="motorFixtVOffset"	value="0.002"/>
+  <xacro:property name="motorFixtHLength" 	value="0.040"/>
+  <xacro:property name="motorFixtHWidth" 	value="0.040"/>
   <xacro:property name="motorFixtHHeigth" 	value="0.003"/>
   <xacro:property name="motorFixtHMass" 	value="1"/>
-  <xacro:property name="cameraSize" 	value="0.02"/>
-  <xacro:property name="cameraMass" 	value="0.5"/>
+  <xacro:property name="casterRadius" 	value="0.02"/>
+  <xacro:property name="camLength" 	value="0.02"/>
+  <xacro:property name="camWidth" 	value="0.02"/>
+  <xacro:property name="camHeigth" 	value="0.02"/>
+  <xacro:property name="camMass" 	value="0.5"/>
+  <xacro:property name="camPitch" 	value="0.3"/>
+  <xacro:property name="camXOffset" 	value="0.175"/>
+  <xacro:property name="camYOffset" 	value="0.05"/>
+  <xacro:property name="lidarBaseRadius" 	value="0.035"/>
+  <xacro:property name="lidarBaseLength" 	value="0.035"/>
+  <xacro:property name="lidarBaseMass" 		value="0.5"/>
+  <xacro:property name="lidarBaseXOffset" 	value="0.14"/>
+  <xacro:property name="lidarHeadRadius" 	value="0.035"/>
+  <xacro:property name="lidarHeadLength" 	value="0.020"/>
+  <xacro:property name="lidarHeadMass" 		value="0.5"/>
+  <xacro:property name="imuLength" 	value="0.010"/>
+  <xacro:property name="imuWidth" 	value="0.005"/>
+  <xacro:property name="imuHeigth" 	value="0.010"/>
+  <xacro:property name="imuMass" 	value="1"/>
   <xacro:include filename="$(find twirtee_description)/urdf/materials.xacro" />
   <xacro:include filename="$(find twirtee_description)/urdf/macros.xacro" />
@@ -57,25 +81,28 @@
 <!-- =========================== -->
   <link name="footprint" />
-<!-- Level 0 -->
+<!-- floor 0 -->
   <joint name="base_joint" type="fixed">
     <parent link="footprint"/>
-    <child link="level0"/>
-      <origin xyz="0 0 ${wheelRadius+wheelFloor0Offset+floor0Heigth/2}" rpy="0 0 0" />
-  </joint>
-  <link name="level0">
+    <child link="floor0"/>
+      <origin xyz="0 0 ${wheelRadius+wheelOffset+motorFixtVOffset+motorFixtVLength/2.0+motorFixtHHeigth+floor0Heigth/2.0}" rpy="0 0 0" />
+  </joint>
+  <link name="floor0">
     <visual>
       <geometry>
 		<box size="${floor0Length} ${floor0Width} ${floor0Heigth}" />
-	    <cylinder radius="${spacerRadius}" length="${spacer01Width}"/>
-      </geometry>
-    </visual>
-  </link>
-<!-- Level 1 -->
-  <joint name="l0l1_joint" type="fixed">
-    <parent link="level0"/>
-    <child link="level1"/>
+      </geometry>
+    </visual>
+	<f0Pilar tX="-1.0" tY="-1.0" />
+	<f0Pilar tX="1.0" tY="-1.0" />
+	<f0Pilar tX="-1.0" tY="1.0" />
+	<f0Pilar tX="1.0" tY="1.0" />
+  </link>
+<!-- floor 1 -->
+  <joint name="f0f1_joint" type="fixed">
+    <parent link="floor0"/>
+    <child link="floor1"/>
 	<origin xyz=" 0.0 0.0 ${spacer01Width+floor1Heigth/2}" rpy="0 0 0" />
   </joint>
-  <link name="level1">
+  <link name="floor1">
     <visual>
       <origin xyz="0 0 0" rpy="0 0 0" />
@@ -84,12 +111,16 @@
       </geometry>
     </visual>
-  </link>
-<!-- Level 2 -->
-  <joint name="l1l2_joint" type="fixed">
-    <parent link="level1"/>
-    <child link="level2"/>
+	<f1Pilar tX="-1.0" tY="-1.0" />
+	<f1Pilar tX="1.0" tY="-1.0" />
+	<f1Pilar tX="-1.0" tY="1.0" />
+	<f1Pilar tX="1.0" tY="1.0" />
+  </link>
+<!-- floor 2 -->
+  <joint name="f1f2_joint" type="fixed">
+    <parent link="floor1"/>
+    <child link="floor2"/>
 	<origin xyz=" 0.0 0.0 ${spacer12Width+floor1Heigth/2}" rpy="0 0 0" />
   </joint>
-  <link name="level2">
+  <link name="floor2">
     <visual>
       <origin xyz="0 0 0" rpy="0 0 0" />
@@ -104,15 +135,81 @@
 <wheel lr="left" tY="1"/>
 <wheel lr="right" tY="-1"/>
+<caster lr="left" tY="1"/>
+<caster lr="right" tY="-1"/>
 <!-- ========================== -->
 <!--          MOTORS            -->
 <!-- ========================== -->
+<motor lr="left" tY="1"/>
+<motor lr="right" tY="-1"/>
 <!-- ========================== -->
 <!--          CAMERA            -->
 <!-- ========================== -->
+  <joint name="f2_cam_joint" type="fixed">
+    <parent link="floor2"/>
+    <child link="cam"/>
+	<origin xyz=" ${camXOffset} ${camYOffset} ${floor2Heigth/2+camHeigth/2.0+0.02}" rpy="0 ${camPitch} 0" />
+  </joint>
+  <link name="cam">
+    <visual>
+      <origin xyz="0 0 0" rpy="0 0 0" />
+      <geometry>
+		<box size="${camLength} ${camWidth} ${camHeigth}" />
+      </geometry>
+	  <material name="orange">
+		  <color rgba="${255/255} ${108/255} ${10/255} 1.0"/>
+	  </material>
+    </visual>
+  </link>
 <!-- ========================== -->
 <!--          IMU            -->
 <!-- ========================== -->
+  <joint name="f1_imu_joint" type="fixed">
+    <parent link="floor1"/>
+    <child link="imu"/>
+	<origin xyz=" 0.0 0.0 ${floor1Heigth/2+imuHeigth/2.0}" rpy="0 0 0" />
+  </joint>
+  <link name="imu">
+    <visual>
+      <origin xyz="0 0 0" rpy="0 0 0" />
+      <geometry>
+		<box size="${imuLength} ${imuWidth} ${imuHeigth}" />
+      </geometry>
+	  <material name="orange">
+		  <color rgba="${255/255} ${108/255} ${10/255} 1.0"/>
+	  </material>
+    </visual>
+  </link>
 <!-- ========================= -->
 <!--           LIDAR           -->
 <!-- ========================= -->
+  <joint name="f2_lidarbase_joint" type="fixed">
+    <parent link="floor2"/>
+    <child link="lidarbase"/>
+	<origin xyz=" ${lidarBaseXOffset} 0.0 ${floor2Heigth/2+lidarBaseLength/2.0}" rpy="0 0 0" />
+  </joint>
+  <link name="lidarbase">
+    <visual>
+      <origin xyz="0 0 0" rpy="0 0 0" />
+      <geometry>
+		<cylinder radius="${lidarBaseRadius}" length="${lidarBaseLength}" />
+      </geometry>
+    </visual>
+  </link>
+  <joint name="lidarbase_head_joint" type="continuous">
+	<axis xyz="0.0 0.0 1.0" />
+    <parent link="lidarbase"/>
+    <child link="lidarhead"/>
+	<origin xyz=" 0.0 0.0 ${lidarBaseLength/2.0+lidarHeadLength/2.0}" rpy="0 0 0" />
+  </joint>
+  <link name="lidarhead">
+    <visual>
+      <origin xyz="0 0 0" rpy="0 0 0" />
+      <geometry>
+		<cylinder radius="${lidarHeadRadius}" length="${lidarHeadLength}"/>
+      </geometry>
+	  <material name="brown">
+		  <color rgba="${222/255} ${207/255} ${195/255} 1.0"/>
+	  </material>
+    </visual>
+  </link>
 </robot>
